Commit message: Full Robot Spawner in Gazebo Fortress

File: ros2_ws/src/wetexplorer/wetexplorer_description/urdf/accesories/linear_actuator.xacro (robot description, xacro)
@@ -116,11 +116,11 @@
         rpy="0 0 0" />
       <mass
-        value="0.14496084881217" />
-      <inertia
-        ixx="0.000997897349092488"
-        ixy="1.17400522028665E-13"
-        ixz="-1.40067550336596E-11"
-        iyy="0.000997913372548"
-        iyz="1.27630788642497E-11"
+        value="0.25" />
+      <inertia
+        ixx="0.00997897349092488"
+        ixy="1.17400522028665E-6"
+        ixz="-1.40067550336596E-6"
+        iyy="0.00997913372548"
+        iyz="1.27630788642497E-6"
         izz="0.01" />
     </inertial>

File: ros2_ws/src/wetexplorer/wetexplorer_description/urdf/chassis_static.xacro (robot description, xacro)
@@ -191,5 +191,5 @@
       </collision> -->
     </link>
-    <joint name="pulleys_right_link"
+    <joint name="pulleys_left_joint"
       type="fixed">
       <origin
@@ -332,5 +332,5 @@
       </collision> -->
     </link>
-    <joint name="pulley_support_right_link"
+    <joint name="pulley_support_right_joint"
       type="fixed">
       <origin
