Commit message: Migration of robot description

File: ros2_ws/src/wetexplorer/wetexplorer_description/urdf/accesories/aluminium_frame.xacro (robot description, xacro)
@@ -23,5 +23,5 @@
       <geometry>
         <mesh
-          filename="package://wetexplorer_description/meshes/extra/aluminium_frame_link.STL" />
+          filename="package://wetexplorer_description/meshes/WETExplorer/gas_analyzer_support_link.STL" />
       </geometry>
       <material
@@ -37,5 +37,5 @@
       <geometry>
         <mesh
-          filename="package://wetexplorer_description/meshes/extra/aluminium_frame_link.STL" />
+          filename="package://max_light_pkg/meshes/extra/aluminium_frame_link.STL" />
       </geometry>
     </collision> -->

File: ros2_ws/src/wetexplorer/wetexplorer_description/urdf/chassis_static.xacro (robot description, xacro)
@@ -1,5 +1,5 @@
 <?xml version="1.0" encoding="utf-8"?>
 <robot xmlns:xacro="http://www.ros.org/wiki/xacro" name="maxii">
-    <!-- Define materials EOOO -->
+  <!-- Define materials EOOO -->
     <material name="green">
        <color rgba="0 1 0 1.0"/>
@@ -108,22 +108,4 @@
         xyz="0 1 0" />
     </joint>
-    <transmission name="trans_right_sprocket">
-        <type>transmission_interface/SimpleTransmission</type>
-        <joint name="power_pulley_right_joint">
-        <hardwareInterface>hardware_interface/VelocityJointInterface</hardwareInterface>
-        </joint>
-        <actuator name="motor_right_sprocket">
-        <mechanicalReduction>100</mechanicalReduction>
-        </actuator>
-    </transmission>
-    <gazebo reference="right_sprocket">
-        <gravity>true</gravity>
-        <mu1>0.5</mu1>
-        <mu2>0.5</mu2>
-        <kd>10</kd>
-        <kp>10000000000.0</kp>
-        <fdir1>0 0 1</fdir1>
-        <selfCollide>false</selfCollide>
-    </gazebo>
     <link name="power_pulley_left_link">
       <inertial>
@@ -174,141 +156,4 @@
         xyz="0 1 0" />
     </joint>
-    <transmission name="trans_left_sprocket">
-        <type>transmission_interface/SimpleTransmission</type>
-        <joint name="power_pulley_left_joint">
-        <hardwareInterface>hardware_interface/VelocityJointInterface</hardwareInterface>
-        </joint>
-        <actuator name="motor_left_sprocket">
-        <mechanicalReduction>100</mechanicalReduction>
-        </actuator>
-    </transmission>
-    <gazebo reference="left_sprocket">
-        <gravity>true</gravity>
-        <mu1>0.5</mu1>
-        <mu2>0.5</mu2>
-        <kd>10</kd>
-        <kp>10000000000.0</kp>
-        <fdir1>0 0 1</fdir1>
-        <selfCollide>false</selfCollide>
-    </gazebo>
-    <link
-      name="track_left_link">
-      <inertial>
-        <origin
-          xyz="-0.0001779 0.3045 -0.043666"
-          rpy="0 0 0" />
-        <mass
-          value="3" />
-        <inertia
-          ixx="0.094232"
-          ixy="-1.3409E-17"
-          ixz="0.025653"
-          iyy="0.34414"
-          iyz="7.2097E-18"
-          izz="0.26251" />
-      </inertial>
-      <visual>
-        <origin
-          xyz="0 0 0"
-          rpy="0 0 0" />
-        <geometry>
-          <mesh
-            filename="package://wetexplorer_description/meshes/WETExplorer/track_left_link.STL" />
-        </geometry>
-        <material name="black"/>
-      </visual>
-      <collision>
-        <origin
-          xyz="0 0 0"
-          rpy="0 0 0" />
-        <geometry>
-          <mesh
-            filename="package://wetexplorer_description/meshes/WETExplorer/track_left_link.STL" />
-        </geometry>
-      </collision>
-    </link>
-    <joint name="track_left_joint"
-      type="revolute">
-      <origin
-        xyz="0 0 0"
-        rpy="0 0 0" />
-      <parent
-        link="base_link" />
-      <child
-        link="track_left_link" />
-      <axis
-        xyz="0 0 0" />
-      "<limit velocity="6.5" effort="1000" lower="0" upper="0" />"
-    </joint>
-    <gazebo reference="track_left_link">
-        <disableFixedJointLumping>true</disableFixedJointLumping>
-        <preserveFixedJoint>true</preserveFixedJoint>
-        <gravity>true</gravity>
-        <mu1>0.3</mu1>
-        <mu2>0.5</mu2>
-        <kd>1</kd>
-        <kp>10000000000.0</kp>
-        <fdir1>0 1 0</fdir1>
-        <selfCollide>false</selfCollide>
-    </gazebo>
-    <link name="track_right_link">
-      <inertial>
-        <origin
-          xyz="-0.0001779 -0.3045 -0.043666"
-          rpy="0 0 0" />
-        <mass
-          value="3" />
-        <inertia
-          ixx="0.094231632"
-          ixy="-6.3364E-18"
-          ixz="0.025652857"
-          iyy="0.344135139"
-          iyz="-4.0857E-18"
-          izz="0.262511007" />
-      </inertial>
-      <visual>
-        <origin
-          xyz="0 0 0"
-          rpy="0 0 0" />
-        <geometry>
-          <mesh
-            filename="package://wetexplorer_description/meshes/WETExplorer/track_right_link.STL" />
-        </geometry>
-        <material name="black"/>
-      </visual>
-      <collision>
-        <origin
-          xyz="0 0.0 0"
-          rpy="0 0 0" />
-        <geometry>
-          <mesh
-            filename="package://wetexplorer_description/meshes/WETExplorer/track_right_link.STL" />
-        </geometry>
-      </collision>
-    </link>
-    <joint name="track_right_joint"
-      type="revolute">
-      <origin
-        xyz="0 0 0"
-        rpy="0 0 0" />
-      <parent
-        link="base_link" />
-      <child
-        link="track_right_link" />
-      <axis
-        xyz="0 0 0" />
-      "<limit velocity="6.5" effort="1000" lower="0" upper="0" />"
-    </joint>
-    <gazebo reference="track_right_link">
-        <disableFixedJointLumping>true</disableFixedJointLumping>
-        <preserveFixedJoint>true</preserveFixedJoint>
-        <gravity>true</gravity>
-        <mu1>0.3</mu1>
-        <mu2>0.5</mu2>
-        <kd>1</kd>
-        <kp>10000000000.0</kp>
-        <fdir1>0 1 0</fdir1>
-        <selfCollide>false</selfCollide>
-    </gazebo>
     <link name="pulleys_left_link">
       <inertial>
@@ -498,67 +343,4 @@
       <axis
         xyz="0 0 0" />
-    </joint>
-    <!-- Control -->
-    <!-- Gazebo plugin for ROS Control -->
-    <gazebo reference="chassis_link">
-      <material>Gazebo/Green</material>
-    </gazebo>
-    <gazebo reference="pulleys_right_link">
-      <material>Gazebo/Grey</material>
-    </gazebo>
-    <gazebo reference="pulleys_left_link">
-      <material>Gazebo/Grey</material>
-    </gazebo>
-    <gazebo reference="power_pulley_left_link">
-      <material>Gazebo/Grey</material>
-    </gazebo>
-    <gazebo reference="power_pulley_right_link">
-      <material>Gazebo/Grey</material>
-    </gazebo>
-    <gazebo reference="track_left_link">
-      <material>Gazebo/DarkGrey</material>
-    </gazebo>
-    <gazebo reference="track_right_link">
-      <material>Gazebo/DarkGrey</material>
-    </gazebo>
-    <gazebo reference="pulley_support_left_link">
-      <material>Gazebo/Red</material>
-    </gazebo>
-    <gazebo reference="pulley_support_right_link">
-      <material>Gazebo/Red</material>
-    </gazebo>
-    <gazebo>
-      <plugin filename="libSimpleTrackedVehiclePlugin.so" name="simple_tracked_vehicle">
-        <body>base_link</body>
-        <left_track>track_left_link</left_track>
-        <right_track>track_right_link</right_track>
-        <steering_efficiency>0.6</steering_efficiency>
-        <tracks_separation>0.6108</tracks_separation>
-        <max_velocity>1.5</max_velocity>
-        <max_acceleration>1.4</max_acceleration>
-        <track_mu>1.0</track_mu>
-        <track_mu2>0.5</track_mu2>
-      </plugin>
-      <gui>
-          <plugin name="keyboard" filename="libKeyboardGUIPlugin.so"/>
-      </gui>
-      <plugin filename="libKeysToCmdVelPlugin.so" name="keyboard_control">
-          <publish_as_twist>true</publish_as_twist>
-          <cmd_vel_topic>~/WetExplorer/cmd_vel_twist</cmd_vel_topic>
-      </plugin>
-        <!-- setup of the interface -->
-      <plugin name='tracked_vehicle_interface' filename='libgazebo_ros_tracked_vehicle_interface.so'>
-        <commandROSTopic>/WetExplorer/cmd_vel</commandROSTopic>
-        <commandIGNTopic>~/WetExplorer/cmd_vel_twist</commandIGNTopic>
-        <!-- <odometryTopic>~odom</odometryTopic>    -->
-        <trackSpeedTopic>~/WetExplorer/track_speed</trackSpeedTopic>  <!-- gazebo topic of SimpleTrackedVehicle -->
-        <robotBaseFrame>base_link</robotBaseFrame>
-        <odometryFrame>gazebo_odom</odometryFrame>
-        <tracks_separation>0.6108</tracks_separation>
-        <publishOdomTF>False</publishOdomTF>
-        <updateRate>50.0</updateRate>
-        <!-- <odometrySource>encoder</odometrySource> --> <!-- [encoder,world] - choose world for ground truth -->
-      </plugin>
-    </gazebo>
-  </xacro:macro>
+    </joint><!-- Define materials EOOO -->
 </robot>

Commit message: Updated Description and mesh folder cleanup

File: ros2_ws/src/wetexplorer/wetexplorer_description/urdf/accesories/aluminium_frame.xacro (robot description, xacro)
@@ -23,5 +23,5 @@
       <geometry>
         <mesh
-          filename="package://wetexplorer_description/meshes/WETExplorer/gas_analyzer_support_link.STL" />
+          filename="package://wetexplorer_description/meshes/gas_analyzer_support_link.STL" />
       </geometry>
       <material

File: ros2_ws/src/wetexplorer/wetexplorer_description/urdf/accesories/central_frame.xacro (robot description, xacro)
@@ -23,5 +23,5 @@
       <geometry>
         <mesh
-          filename="package://wetexplorer_description/meshes/WETExplorer/central_frame_link.STL" />
+          filename="package://wetexplorer_description/meshes/central_frame_link.STL" />
       </geometry>
       <material

File: ros2_ws/src/wetexplorer/wetexplorer_description/urdf/accesories/gas_analyzer.xacro (robot description, xacro)
@@ -22,5 +22,5 @@
       <geometry>
         <mesh
-          filename="package://wetexplorer_description/meshes/WETExplorer/gas_analyzer_link.STL" />
+          filename="package://wetexplorer_description/meshes/gas_analyzer_link.STL" />
       </geometry>
       <material
@@ -73,5 +73,5 @@
         <geometry>
           <mesh
-            filename="package://wetexplorer_description/meshes/WETExplorer/gas_analyzer_support_link.STL" />
+            filename="package://wetexplorer_description/meshes/gas_analyzer_support_link.STL" />
         </geometry>
         <material

File: ros2_ws/src/wetexplorer/wetexplorer_description/urdf/accesories/gps.xacro (robot description, xacro)
@@ -22,5 +22,5 @@
       <geometry>
         <mesh
-          filename="package://wetexplorer_description/meshes/WETExplorer/gps_frame_link.STL" />
+          filename="package://wetexplorer_description/meshes/gps_frame_link.STL" />
       </geometry>
       <material
@@ -74,5 +74,5 @@
       <geometry>
         <mesh
-          filename="package://wetexplorer_description/meshes/WETExplorer/gps_link.STL" />
+          filename="package://wetexplorer_description/meshes/gps_link.STL" />
       </geometry>
       <material

File: ros2_ws/src/wetexplorer/wetexplorer_description/urdf/accesories/imu.xacro (robot description, xacro)
@@ -46,8 +46,7 @@
     <sensor name="imu_sensor" type="imu">
       <always_on>1</always_on>
-      <bodyName>imu_link</bodyName>
-      <update_rate>250.0</update_rate>
+      <update_rate>1</update_rate>
       <visualize>true</visualize>
-      <topic>imu/data</topic>
+      <topic>imu</topic>
     </sensor>
     <!-- <plugin name="imu_controller" filename="libhector_gazebo_ros_imu.so">

File: ros2_ws/src/wetexplorer/wetexplorer_description/urdf/accesories/linear_actuator.xacro (robot description, xacro)
@@ -23,5 +23,5 @@
       <geometry>
         <mesh
-          filename="package://wetexplorer_description/meshes/WETExplorer/linear_actuator_support_link.STL" />
+          filename="package://wetexplorer_description/meshes/linear_actuator_support_link.STL" />
       </geometry>
       <material
@@ -131,5 +131,5 @@
       <geometry>
         <mesh
-          filename="package://wetexplorer_description/meshes/WETExplorer/prismatic_link.STL" />
+          filename="package://wetexplorer_description/meshes/prismatic_link.STL" />
       </geometry>
       <material
@@ -203,5 +203,5 @@
       <geometry>
         <mesh
-          filename="package://wetexplorer_description/meshes/WETExplorer/coupling_link.STL" />
+          filename="package://wetexplorer_description/meshes/coupling_link.STL" />
       </geometry>
       <material
@@ -217,5 +217,5 @@
       <geometry>
         <mesh
-          filename="package://wetexplorer_description/meshes/WETExplorer/coupling_link.STL" />
+          filename="package://wetexplorer_description/meshes/coupling_link.STL" />
       </geometry>
     </collision>
@@ -256,5 +256,5 @@
       <geometry>
         <mesh
-          filename="package://wetexplorer_description/meshes/WETExplorer/chamber_holder_link.STL" />
+          filename="package://wetexplorer_description/meshes/chamber_holder_link.STL" />
       </geometry>
       <material
@@ -270,5 +270,5 @@
       <geometry>
         <mesh
-          filename="package://wetexplorer_description/meshes/WETExplorer/chamber_holder_link.STL" />
+          filename="package://wetexplorer_description/meshes/chamber_holder_link.STL" />
       </geometry>
     </collision>
@@ -321,5 +321,5 @@
       <geometry>
         <mesh
-          filename="package://wetexplorer_description/meshes/WETExplorer/chamber_link.STL" />
+          filename="package://wetexplorer_description/meshes/chamber_link.STL" />
       </geometry>
       <material
@@ -335,5 +335,5 @@
       <geometry>
         <mesh
-          filename="package://wetexplorer_description/meshes/WETExplorer/chamber_link.STL" />
+          filename="package://wetexplorer_description/meshes/chamber_link.STL" />
       </geometry>
     </collision>

File: ros2_ws/src/wetexplorer/wetexplorer_description/urdf/chassis_static.xacro (robot description, xacro)
@@ -40,5 +40,5 @@
         <geometry>
           <mesh
-            filename="package://wetexplorer_description/meshes/WETExplorer/base_link.STL" />
+            filename="package://wetexplorer_description/meshes/base_link.STL" />
         </geometry>
         <material name="green"/>
@@ -50,5 +50,5 @@
         <geometry>
           <mesh
-            filename="package://wetexplorer_description/meshes/WETExplorer/base_link.STL" />
+            filename="package://wetexplorer_description/meshes/base_link.STL" />
         </geometry>
       </collision>
@@ -81,5 +81,5 @@
         <geometry>
           <mesh
-            filename="package://wetexplorer_description/meshes/WETExplorer/power_pulley_right_link.STL" />
+            filename="package://wetexplorer_description/meshes/power_pulley_right_link.STL" />
         </geometry>
         <material name="grey"/>
@@ -129,5 +129,5 @@
         <geometry>
           <mesh
-            filename="package://wetexplorer_description/meshes/WETExplorer/power_pulley_left_link.STL" />
+            filename="package://wetexplorer_description/meshes/power_pulley_left_link.STL" />
         </geometry>
         <material name="grey"/>
@@ -177,5 +177,5 @@
         <geometry>
           <mesh
-            filename="package://wetexplorer_description/meshes/WETExplorer/pulleys_left_link.STL" />
+            filename="package://wetexplorer_description/meshes/pulleys_left_link.STL" />
         </geometry>
         <material name="grey"/>
@@ -224,5 +224,5 @@
         <geometry>
           <mesh
-            filename="package://wetexplorer_description/meshes/WETExplorer/pulleys_right_link.STL" />
+            filename="package://wetexplorer_description/meshes/pulleys_right_link.STL" />
         </geometry>
         <material name="grey"/>
@@ -271,5 +271,5 @@
         <geometry>
           <mesh
-            filename="package://wetexplorer_description/meshes/WETExplorer/pulley_support_left_link.STL" />
+            filename="package://wetexplorer_description/meshes/pulley_support_left_link.STL" />
         </geometry>
         <material name="red"/>
@@ -318,5 +318,5 @@
         <geometry>
           <mesh
-            filename="package://wetexplorer_description/meshes/WETExplorer/pulley_support_right_link.STL" />
+            filename="package://wetexplorer_description/meshes/pulley_support_right_link.STL" />
         </geometry>
         <material name="red"/>

File: ros2_ws/src/wetexplorer/wetexplorer_description/urdf/tracks/tracks_static.xacro (robot description, xacro)
@@ -27,7 +27,13 @@
         <material name="black"/>
       </visual>
+      <collision>
+          <geometry>
+            <mesh
+              filename="package://wetexplorer_description/meshes/track_left_link.STL" />
+          </geometry>
+        </collision>
     </link>
     <joint name="track_left_joint"
-      type="fixed">
+      type="revolute">
       <origin
         xyz="0 0 0"
@@ -37,4 +43,7 @@
       <child
         link="track_left_link" />
+      <axis
+        xyz="0 1 0" />
+      <limit velocity="6.5" effort="1000" lower="0" upper="0" />
     </joint>
     <link name="track_right_link">
@@ -63,7 +72,13 @@
         <material name="black"/>
       </visual>
+      <collision>
+          <geometry>
+            <mesh
+              filename="package://wetexplorer_description/meshes/track_right_link.STL" />
+          </geometry>
+      </collision>
     </link>
     <joint name="track_right_joint"
-      type="fixed">
+      type="revolute">
       <origin
         xyz="0 0 0"
@@ -73,4 +88,27 @@
       <child
         link="track_right_link" />
+      <axis
+        xyz="0 1 0" />
+      <limit velocity="6.5" effort="1000" lower="0" upper="0" />
     </joint>
+    <gazebo>
+      <plugin name="gz::sim::systems::TrackedVehicle" filename="gz-sim-tracked-vehicle-system">
+        <body>base_link</body>
+        <left_track><link>track_left_link</link></left_track>
+        <right_track><link>track_right_link</link></right_track>
+        <tracks_separation>0.6108</tracks_separation>
+        <tracks_height>0.18094</tracks_height>
+        <steering_efficiency>0.5</steering_efficiency>
+      </plugin>
+      <plugin name='gz::sim::systems::TrackController' filename='gz-sim-track-controller-system'>
+          <link>track_left_link</link>
+          <min_velocity>-1.0</min_velocity>
+          <max_velocity>1.0</max_velocity>
+      </plugin>
+      <plugin name='gz::sim::systems::TrackController' filename='gz-sim-track-controller-system'>
+          <link>track_right_link</link>
+          <min_velocity>-1.0</min_velocity>
+          <max_velocity>1.0</max_velocity>
+      </plugin>
+    </gazebo>
 </robot>
