Commit message: Add Updated Model: Description of the latest wetexplorer model including the 2 depth cameras and new lifting mechanism

File: ros2_ws/src/wetexplorer/wetexplorer_description/urdf/accesories/gas_analyzer.xacro (robot description, xacro)
@@ -4,15 +4,15 @@
     <inertial>
       <origin
-        xyz="-0.18424 -1.1028E-14 0.27892"
+        xyz="-0.160926382849307 -6.27116167484449E-15 0.278920978379107"
         rpy="0 0 0" />
       <mass
-        value="21" />
+        value="60.1217120629733" />
       <inertia
-        ixx="0.870247786"
-        ixy="-4.0644E-17"
-        ixz="-5.0732E-14"
-        iyy="0.508970755"
-        iyz="2.2193E-06"
-        izz="1.267160807" />
+        ixx="0.702337674386062"
+        ixy="-5.14331673511432E-17"
+        ixz="-5.0757869374301E-14"
+        iyy="1.45715235750158"
+        iyz="2.21930158397138E-06"
+        izz="1.83867554764121" />
     </inertial>
     <visual>

File: ros2_ws/src/wetexplorer/wetexplorer_description/urdf/accesories/gps.xacro (robot description, xacro)
@@ -4,15 +4,15 @@
     <inertial>
       <origin
-        xyz="0.105414522198737 1.32321772844421E-15 0.424896531084323"
+        xyz="0.105414522198745 2.11113479880442E-16 0.42142097837912"
         rpy="0 0 0" />
       <mass
-        value="0.43752152687841" />
+        value="0.404841115087331" />
       <inertia
-        ixx="0.0297577743435381"
-        ixy="-2.01741520712827E-16"
-        ixz="6.70399343732719E-17"
-        iyy="0.0015552380426208"
-        iyz="2.0466027135012E-16"
-        izz="0.0282575439845002" />
+        ixx="0.00762661855296656"
+        ixy="-8.51690952924258E-21"
+        ixz="6.70526492376864E-17"
+        iyy="0.00157192564919616"
+        iyz="4.79291022859442E-17"
+        izz="0.00612638819392862" />
     </inertial>
     <visual>
@@ -22,5 +22,5 @@
       <geometry>
         <mesh
-          filename="package://wetexplorer_description/meshes/gps_frame_link.STL" />
+          filename="package://wetexplorer_description/meshes/extra/gps_frame_link.STL" />
       </geometry>
       <material
@@ -56,15 +56,15 @@
     <inertial>
       <origin
-        xyz="-2.64164212384899E-05 -0.549999997401756 -0.0043107897343504"
+        xyz="-2.23672210816483E-05 -0.2865087525775 0.00451065274111317"
         rpy="0 0 0" />
       <mass
-        value="0.200329985591101" />
+        value="0.236596279105962" />
       <inertia
-        ixx="0.000140014066561097"
-        ixy="5.17044736191504E-11"
-        ixz="-3.22977757637025E-08"
-        iyy="0.000136584182993869"
-        iyz="-1.25336110166667E-11"
-        izz="0.000265443361867639" />
+        ixx="0.000153435356186975"
+        ixy="5.16572317628455E-11"
+        ixz="-3.22977757581418E-08"
+        iyy="0.000150409946833309"
+        iyz="-1.25336119132743E-11"
+        izz="0.000290224818991714" />
     </inertial>
     <visual>
@@ -74,5 +74,5 @@
       <geometry>
         <mesh
-          filename="package://wetexplorer_description/meshes/gps_link.STL" />
+          filename="package://wetexplorer_description/meshes/extra/gps_link.STL" />
       </geometry>
       <material
@@ -95,5 +95,5 @@
     type="fixed">
     <origin
-      xyz="0.105414522198752 0.550000000000003 0.521670978379597"
+      xyz="0.10541 0.28651 0.53942"
       rpy="0 0 0" />
     <parent

File: ros2_ws/src/wetexplorer/wetexplorer_description/urdf/accesories/imu.xacro (robot description, xacro)
@@ -1,39 +1,56 @@
 <?xml version="1.0"?>
 <robot xmlns:xacro="http://www.ros.org/wiki/xacro" name="imu">
-  <!-- IMU Link -->
-  <link name="imu_link">
+  <link
+    name="imu_link">
     <inertial>
-      <origin xyz="-0.00144144958218404 8.57757393428608E-05 0.000661614742153149" rpy="0 0 0" />
-      <mass value="0.00959464796722065" />
+      <origin
+        xyz="0.0055655602260675 -0.00292820256170392 -0.00130118633552501"
+        rpy="0 0 0" />
+      <mass
+        value="0.0218886437543552" />
       <inertia
-        ixx="1.30281027931082E-06"
-        ixy="-1.56746685836304E-11"
-        ixz="4.93823028160914E-11"
-        iyy="1.27869196687108E-06"
-        iyz="-6.22065563257926E-09"
-        izz="2.51111665492873E-06" />
+        ixx="4.619031605549E-06"
+        ixy="6.09459742090583E-07"
+        ixz="-6.70691041223252E-07"
+        iyy="3.90481536378184E-06"
+        iyz="3.27283112860456E-07"
+        izz="6.9165264373137E-06" />
     </inertial>
     <visual>
-      <origin xyz="0 0 0" rpy="0 0 0" />
+      <origin
+        xyz="0 0 0"
+        rpy="0 0 0" />
       <geometry>
-        <mesh filename="package://wetexplorer_description/meshes/extra/imu_link.STL" />
+        <mesh
+          filename="package://wetexplorer_description/meshes/imu_link.STL" />
       </geometry>
-      <material name="">
-        <color rgba="0.752941176470588 0.752941176470588 0.752941176470588 1" />
+      <material
+        name="">
+        <color
+          rgba="0.752941176470588 0.752941176470588 0.752941176470588 1" />
       </material>
     </visual>
-    <!-- <collision>
-      <origin xyz="0 0 0" rpy="0 0 0" />
+    <collision>
+      <origin
+        xyz="0 0 0"
+        rpy="0 0 0" />
       <geometry>
-        <mesh filename="package://wetexplorer_description/meshes/extra/imu_link.STL" />
+        <mesh
+          filename="package://wetexplorer_description/meshes/imu_link.STL" />
       </geometry>
-    </collision> -->
+    </collision>
   </link>
-  <!-- IMU Joint -->
-  <joint name="imu_joint" type="fixed">
-    <origin xyz="0.00278 0 0.16463" rpy="0 0 0" />
-    <parent link="base_link" />
-    <child link="imu_link" />
-    <axis xyz="0 0 1" />
+  <joint
+    name="imu_joint"
+    type="fixed">
+    <origin
+      xyz="0.06745 0 0.16966"
+      rpy="0 0 0" />
+    <parent
+      link="base_link" />
+    <child
+      link="imu_link" />
+    <axis
+      xyz="0 0 0" />
   </joint>
   <gazebo reference="imu_link">

File: ros2_ws/src/wetexplorer/wetexplorer_description/urdf/chassis_static.xacro (robot description, xacro)
@@ -60,5 +60,5 @@
         <axis xyz="0 0 0"/>
     </joint>
-    <link name="power_pulley_right_link">
+    <link name="sprocket_right_link">
       <inertial>
         <origin
@@ -96,5 +96,5 @@
     </link>
       <joint
-      name="power_pulley_right_joint"
+      name="sprocket_right_joint"
       type="continuous">
       <origin
@@ -104,9 +104,9 @@
         link="base_link" />
       <child
-        link="power_pulley_right_link" />
+        link="sprocket_right_link" />
       <axis
         xyz="0 1 0" />
     </joint>
-    <link name="power_pulley_left_link">
+    <link name="sprocket_left_link">
       <inertial>
         <origin
@@ -144,5 +144,5 @@
     </link>
     <joint
-      name="power_pulley_left_joint"
+      name="sprocket_left_joint"
       type="continuous">
       <origin
@@ -152,5 +152,5 @@
         link="base_link" />
       <child
-        link="power_pulley_left_link" />
+        link="sprocket_left_link" />
       <axis
         xyz="0 1 0" />

File: ros2_ws/src/wetexplorer/wetexplorer_description/urdf/tracks.xacro (robot description, xacro)
@@ -1,5 +1,5 @@
 <?xml version="1.0" encoding="utf-8"?>
 <robot xmlns:xacro="http://www.ros.org/wiki/xacro" name="Wetexplorer">
-  <xacro:include filename="$(find wetexplorer_description)/urdf/camera.xacro" />
+  <!-- <xacro:include filename="$(find wetexplorer_description)/urdf/camera.xacro" /> -->
   <xacro:include filename="$(find wetexplorer_description)/urdf/cylinder_inertia.xacro" />
   <xacro:include filename="$(find wetexplorer_description)/urdf/chassis_static.xacro" />
@@ -13,4 +13,9 @@
   <xacro:include filename="$(find wetexplorer_description)/urdf/front_wheel.xacro"/>
   <xacro:include filename="$(find wetexplorer_description)/urdf/wheel_controller.xacro"/>
+  <xacro:include filename="$(find wetexplorer_description)/urdf/accesories/lift_frame.xacro"/>
+  <xacro:include filename="$(find wetexplorer_description)/urdf/camera1.xacro"/>
+  <xacro:include filename="$(find wetexplorer_description)/urdf/camera2.xacro"/>
+  <xacro:include filename="$(find wetexplorer_description)/urdf/gazebo.xacro"/>
+  <xacro:include filename="$(find wetexplorer_description)/urdf/lift_mechanism.xacro"/>
   <xacro:property name="mu" value="0.7"/>
   <xacro:property name="position_left" value="0.3054"/>
