Commit message: Fix IMU Orientation: now it matches the sensor in real life

File: ros2_ws/src/wetexplorer/wetexplorer_description/urdf/accesories/imu.xacro (robot description, xacro)
@@ -2,5 +2,5 @@
 <robot xmlns:xacro="http://www.ros.org/wiki/xacro" name="imu">
   <link
-    name="imu_link">
+    name="imu_link_target">
     <inertial>
       <origin
@@ -42,5 +42,5 @@
   </link>
   <joint
-    name="imu_joint"
+    name="imu_joint_target"
     type="fixed">
     <origin
@@ -50,9 +50,25 @@
       link="base_link" />
     <child
+      link="imu_link_target" />
+    <axis
+      xyz="0 0 0" />
+  </joint>
+  <link
+    name="imu_link">
+  </link>
+  <joint
+    name="imu_joint"
+    type="fixed">
+    <origin
+      xyz="0.06745 0 0.16966"
+      rpy="-3.141592654 0 0" />
+    <parent
+      link="base_link" />
+    <child
       link="imu_link" />
     <axis
       xyz="0 0 0" />
   </joint>
-  <gazebo reference="imu_link">
+  <gazebo reference="imu_link_target">
       <material>Gazebo/Grey</material>
       <sensor name="imu_sensor" type="imu">
