Commit message: Add TCP Link: RVIZ display and description files updated

File: ros2_ws/src/wetexplorer/wetexplorer_description/urdf/accesories/chamber.xacro (robot description, xacro)
@@ -5,5 +5,5 @@
   <xacro:property name="radius" value="0.015" />
   <xacro:property name="length" value="0.2" />
-  <link name="chamber_link">
+  <link name="tcp_frame">
       <inertial>
           <origin xyz="0 0 0"/>
@@ -24,4 +24,5 @@
       </visual>
   </link>
+  <link name="chamber_link">
   <joint name="chamber_joint"
     type="prismatic">
@@ -32,5 +33,5 @@
       link="base_link" />
     <child
-      link="chamber_link" />
+      link="tcp_frame" />
     <axis
       xyz="0 0 1" />
@@ -41,4 +42,16 @@
       velocity="0.2" />
     <dynamics damping="3.0" friction="0.3"/>
+  </joint>
+  <joint name="chamber_fixed_joint"
+    type="fixed">
+    <origin
+      xyz="0.48712 0 0.00"
+      rpy="0 0 0" />
+    <parent
+      link="base_link" />
+    <child
+      link="chamber_link" />
+    <axis
+      xyz="0 0 1" />
   </joint>
   <transmission name="chamber_transmission">
@@ -101,5 +114,5 @@
   <joint name="chamber_joint_2" type="revolute">
     <origin xyz="0 0 -0.1" rpy="0 0 0" />
-    <parent link="chamber_link" />
+    <parent link="tcp_frame" />
     <child link="chamber_link_2" />
     <axis xyz="1 0 0" />

File: ros2_ws/src/wetexplorer/wetexplorer_description/urdf/camera1.xacro (robot description, xacro)
@@ -101,5 +101,5 @@
           <pose> 0 0 0 0 0 0 </pose>
           <visualize>true</visualize>
-          <update_rate>5</update_rate>
+          <update_rate>15</update_rate>
           <camera>
               <camera_info_topic>camera1/camera_info</camera_info_topic>
@@ -121,5 +121,5 @@
           <pose> 0 0 0 0 0 0 </pose>
           <visualize>true</visualize>
-          <update_rate>5</update_rate>
+          <update_rate>15</update_rate>
           <camera>
               <camera_info_topic>camera1/camera_info</camera_info_topic>

File: ros2_ws/src/wetexplorer/wetexplorer_description/urdf/camera2.xacro (robot description, xacro)
@@ -73,5 +73,5 @@
           <pose> 0 0 0 0 0 0 </pose>
           <visualize>true</visualize>
-          <update_rate>5</update_rate>
+          <update_rate>1</update_rate>
           <camera>
               <camera_info_topic>camera2/camera_info</camera_info_topic>
@@ -93,5 +93,5 @@
           <pose> 0 0 0 0 0 0 </pose>
           <visualize>true</visualize>
-          <update_rate>5</update_rate>
+          <update_rate>1</update_rate>
           <camera>
               <camera_info_topic>camera2/camera_info</camera_info_topic>

File: ros2_ws/src/wetexplorer/wetexplorer_description/urdf/lift_mechanism.xacro (robot description, xacro)
@@ -60,6 +60,29 @@
     <dynamics damping="3.0" friction="0.3"/>
   </joint>
+  <link name="chamber_link">
+  </link>
+  <joint
+    name="chamber_fixed_joint"
+    type="fixed">
+    <origin
+      xyz="0.53912 -0.0001 -0.15"
+      rpy="0 0 0" />
+    <parent
+      link="base_link" />
+    <child
+      link="chamber_link" />
+    <axis
+      xyz="0 0 0" />
+    <limit
+      lower="-0.2"
+      upper="0"
+      effort="100"
+      velocity="0.2" />
+    <dynamics
+      damping="0.05"
+      friction="0.3" />
+  </joint>
   <link
-    name="chamber_link">
+    name="chamber_link_22">
     <inertial>
       <origin
@@ -109,5 +132,5 @@
       link="lift_link" />
     <child
-      link="chamber_link" />
+      link="chamber_link_22" />
     <axis
       xyz="0 0 0" />

File: ros2_ws/src/wetexplorer/wetexplorer_description/urdf/tracks.xacro (robot description, xacro)
@@ -15,5 +15,5 @@
   <xacro:include filename="$(find wetexplorer_description)/urdf/accesories/lift_frame.xacro"/>
   <xacro:include filename="$(find wetexplorer_description)/urdf/camera1.xacro"/>
-  <xacro:include filename="$(find wetexplorer_description)/urdf/camera2.xacro"/>
+  <!-- <xacro:include filename="$(find wetexplorer_description)/urdf/camera2.xacro"/> -->
   <xacro:include filename="$(find wetexplorer_description)/urdf/gazebo.xacro"/>
   <xacro:include filename="$(find wetexplorer_description)/urdf/lift_mechanism.xacro"/>
