Commit message: Add Features: Imu, GPS and Sprocket Sensors added to the model

File: ros2_ws/src/wetexplorer/wetexplorer_description/urdf/accesories/gps.xacro (robot description, xacro)
@@ -109,11 +109,10 @@
   <gazebo reference="gps_link">
       <material>Gazebo/Black</material>
-  </gazebo>
-  <gazebo>
-    <sensor name="navsat_sensor" type="navsat">
-      <always_on>1</always_on>
-      <update_rate>5.0</update_rate>
-      <topic>navsat/fix</topic>
-    </sensor>
+      <sensor name="gps_sensor" type="navsat">
+        <always_on>1</always_on>
+        <update_rate>5.0</update_rate>
+        <topic>navsat/fix</topic>
+        <gz_frame_id>base_link</gz_frame_id>
+      </sensor>
   </gazebo>
 </robot>

File: ros2_ws/src/wetexplorer/wetexplorer_description/urdf/accesories/imu.xacro (robot description, xacro)
@@ -39,15 +39,67 @@
   <gazebo reference="imu_link">
       <material>Gazebo/Grey</material>
+      <sensor name="imu_sensor" type="imu">
+        <always_on>true</always_on>
+        <update_rate>250</update_rate>
+        <enable_orientation>1</enable_orientation>
+        <visualize>true</visualize>
+        <topic>imu/data</topic>
+        <gz_frame_id>base_link</gz_frame_id>
+        <imu>
+          <angular_velocity>
+            <x>
+              <noise type="gaussian">
+                <mean>0.0</mean>
+                <stddev>2e-4</stddev>
+                <bias_mean>0.0000075</bias_mean>
+                <bias_stddev>0.0000008</bias_stddev>
+              </noise>
+            </x>
+            <y>
+              <noise type="gaussian">
+                <mean>0.0</mean>
+                <stddev>2e-4</stddev>
+                <bias_mean>0.0000075</bias_mean>
+                <bias_stddev>0.0000008</bias_stddev>
+              </noise>
+            </y>
+            <z>
+              <noise type="gaussian">
+                <mean>0.0</mean>
+                <stddev>2e-4</stddev>
+                <bias_mean>0.0000075</bias_mean>
+                <bias_stddev>0.0000008</bias_stddev>
+              </noise>
+            </z>
+          </angular_velocity>
+          <linear_acceleration>
+            <x>
+              <noise type="gaussian">
+                <mean>0.0</mean>
+                <stddev>1.7e-2</stddev>
+                <bias_mean>0.1</bias_mean>
+                <bias_stddev>0.001</bias_stddev>
+              </noise>
+            </x>
+            <y>
+              <noise type="gaussian">
+                <mean>0.0</mean>
+                <stddev>1.7e-2</stddev>
+                <bias_mean>0.1</bias_mean>
+                <bias_stddev>0.001</bias_stddev>
+              </noise>
+            </y>
+            <z>
+              <noise type="gaussian">
+                <mean>0.0</mean>
+                <stddev>1.7e-2</stddev>
+                <bias_mean>0.1</bias_mean>
+                <bias_stddev>0.001</bias_stddev>
+              </noise>
+            </z>
+          </linear_acceleration>
+        </imu>
+      </sensor>
   </gazebo>
-  <gazebo>
-    <plugin filename="gz-sim-imu-system"
-        name="gz::sim::systems::Imu">
-    </plugin>
-    <sensor name="imu_sensor" type="imu">
-      <always_on>1</always_on>
-      <update_rate>1</update_rate>
-      <visualize>true</visualize>
-      <topic>imu</topic>
-    </sensor>
     <!-- <plugin name="imu_controller" filename="libhector_gazebo_ros_imu.so">
       <updateRate>250.0</updateRate>
@@ -61,4 +113,3 @@
       <headingGaussianNoise>0.0</headingGaussianNoise>
     </plugin> -->
-  </gazebo>
 </robot>

File: ros2_ws/src/wetexplorer/wetexplorer_description/urdf/front_wheel.xacro (robot description, xacro)
@@ -17,5 +17,5 @@
         <xacro:cylinder_inertia mass="${mass}" radius="${radius}" length="${length}"/>
     </link>
-    <joint name="front_${left_right}_wheel_joint" type="continuous">
+    <joint name="${left_right}_wheel_joint" type="continuous">
         <origin xyz="0.18601 ${position} -0.1259" rpy=" -1.570796 0 0" />
         <parent link="base_link" />
@@ -23,13 +23,4 @@
         <axis  xyz="0 0 1" />
     </joint>
-    <transmission name="trans_front_${left_right}_wheel">
-        <type>transmission_interface/SimpleTransmission</type>
-        <joint name="front_${left_right}_wheel_joint">
-        <hardwareInterface>hardware_interface/EffortJointInterface</hardwareInterface>
-        </joint>
-        <actuator name="motor_front_${left_right}_wheel">
-        <mechanicalReduction>1</mechanicalReduction>
-        </actuator>
-    </transmission>
     <gazebo reference="front_${left_right}_wheel">
         <gravity>true</gravity>

File: ros2_ws/src/wetexplorer/wetexplorer_description/urdf/tracks.xacro (robot description, xacro)
@@ -7,7 +7,15 @@
   <xacro:include filename="$(find wetexplorer_description)/urdf/accesories/aluminium_frame.xacro" />
   <xacro:include filename="$(find wetexplorer_description)/urdf/accesories/central_frame.xacro" />
-  <!-- <xacro:include filename="$(find wetexplorer_description)/urdf/accesories/imu.xacro" />
-  <xacro:include filename="$(find wetexplorer_description)/urdf/accesories/gps.xacro" /> -->
+  <xacro:include filename="$(find wetexplorer_description)/urdf/accesories/imu.xacro" />
+  <xacro:include filename="$(find wetexplorer_description)/urdf/accesories/gps.xacro" /> -
   <xacro:include filename="$(find wetexplorer_description)/urdf/accesories/gas_analyzer.xacro" />
   <!-- <xacro:include filename="$(find wetexplorer_description)/urdf/accesories/linear_actuator.xacro" /> -->
+  <xacro:include filename="$(find wetexplorer_description)/urdf/front_wheel.xacro"/>
+  <xacro:include filename="$(find wetexplorer_description)/urdf/wheel_controller.xacro"/>
+  <xacro:property name="mu" value="0.7"/>
+  <xacro:property name="position_left" value="0.3054"/>
+  <xacro:property name="position_right" value="-0.3054"/>
+  <xacro:front_wheel left_right="left" radius="0.075" length="0.01" position="${position_left}" mu="${mu}"/>
+  <xacro:front_wheel left_right="right" radius="0.075" length="0.01" position="${position_right}" mu="${mu}"/>
+  <xacro:wheel_control name="wheels"/>
 </robot>

Commit message: Fix GPS Plugin

File: ros2_ws/src/wetexplorer/wetexplorer_description/urdf/accesories/gps.xacro (robot description, xacro)
@@ -109,9 +109,47 @@
   <gazebo reference="gps_link">
       <material>Gazebo/Black</material>
-      <sensor name="gps_sensor" type="navsat">
+      <sensor name="gps_sensor" type="gps">
         <always_on>1</always_on>
         <update_rate>5.0</update_rate>
         <topic>navsat/fix</topic>
         <gz_frame_id>base_link</gz_frame_id>
+        <gps>
+          <position_sensing>
+            <horizontal>
+              <noise type="gaussian">
+                <mean>0.0</mean>
+                <stddev>0.00000001</stddev>
+              </noise>
+            </horizontal>
+            <vertical>
+              <noise type="gaussian">
+                <mean>0.0</mean>
+                <stddev>0.00000001</stddev>
+              </noise>
+            </vertical>
+          </position_sensing>
+        </gps>
+      </sensor>
+       <sensor name="gps_sensor_truth" type="gps">
+        <always_on>1</always_on>
+        <update_rate>50.0</update_rate>
+        <topic>gps/ref</topic>
+        <gz_frame_id>base_link</gz_frame_id>
+        <gps>
+          <position_sensing>
+            <horizontal>
+              <noise type="gaussian">
+                <mean>0.0</mean>
+                <stddev>0.0000000</stddev>
+              </noise>
+            </horizontal>
+            <vertical>
+              <noise type="gaussian">
+                <mean>0.0</mean>
+                <stddev>0.0000000</stddev>
+              </noise>
+            </vertical>
+          </position_sensing>
+        </gps>
       </sensor>
   </gazebo>

File: ros2_ws/src/wetexplorer/wetexplorer_description/urdf/accesories/imu.xacro (robot description, xacro)
@@ -134,4 +134,92 @@
         </imu>
       </sensor>
+      <sensor name="imu_sensor_heading" type="imu">
+        <always_on>true</always_on>
+        <update_rate>50</update_rate>
+        <enable_orientation>1</enable_orientation>
+        <visualize>true</visualize>
+        <topic>imu_heading/data</topic>
+        <gz_frame_id>base_link</gz_frame_id>
+        <imu>
+          <angular_velocity>
+            <x>
+              <noise type="gaussian">
+                <mean>0.0</mean>
+                <stddev>0.0</stddev>
+                <bias_mean>0.000001</bias_mean>
+                <bias_stddev>0.000000</bias_stddev>
+              </noise>
+            </x>
+            <y>
+              <noise type="gaussian">
+                <mean>0.0</mean>
+                <stddev>0.0</stddev>
+                <bias_mean>0.000001</bias_mean>
+                <bias_stddev>0.000000</bias_stddev>
+              </noise>
+            </y>
+            <z>
+              <noise type="gaussian">
+                <mean>0.0</mean>
+                <stddev>0.0</stddev>
+                <bias_mean>0.000001</bias_mean>
+                <bias_stddev>0.000000</bias_stddev>
+              </noise>
+            </z>
+          </angular_velocity>
+          <linear_acceleration>
+            <x>
+              <noise type="gaussian">
+                <mean>0.0</mean>
+                <stddev>0.0</stddev>
+                <bias_mean>0.000001</bias_mean>
+                <bias_stddev>0.000000</bias_stddev>
+              </noise>
+            </x>
+            <y>
+              <noise type="gaussian">
+                <mean>0.0</mean>
+                <stddev>0.0</stddev>
+                <bias_mean>0.000001</bias_mean>
+                <bias_stddev>0.000000</bias_stddev>
+              </noise>
+            </y>
+            <z>
+              <noise type="gaussian">
+                <mean>0.0</mean>
+                <stddev>0.0</stddev>
+                <bias_mean>0.000001</bias_mean>
+                <bias_stddev>0.000000</bias_stddev>
+              </noise>
+            </z>
+          </linear_acceleration>
+          <orientation>
+            <x>
+              <noise type="gaussian">
+                <mean>0.0</mean>
+                <stddev>0.0</stddev>
+                <bias_mean>0.000001</bias_mean>
+                <bias_stddev>0.000000</bias_stddev>
+              </noise>
+            </x>
+            <y>
+              <noise type="gaussian">
+                <mean>0.0</mean>
+                <stddev>0.0</stddev>
+                <bias_mean>0.000001</bias_mean>
+                <bias_stddev>0.000000</bias_stddev>
+              </noise>
+            </y>
+            <z>
+              <noise type="gaussian">
+                <mean>0.0</mean>
+                <stddev>0.0</stddev>
+                <bias_mean>0.000001</bias_mean>
+                <bias_stddev>0.000000</bias_stddev>
+              </noise>
+            </z>
+          </orientation>
+        </imu>
+      </sensor>
   </gazebo>
     <!-- <plugin name="imu_controller" filename="libhector_gazebo_ros_imu.so">

File: ros2_ws/src/wetexplorer/wetexplorer_description/urdf/camera1.xacro (robot description, xacro)
@@ -45,5 +45,5 @@
     type="fixed">
     <origin
-      xyz="0.76557 0.117 0.35625"
+      xyz="0.76557 0.117 0.455898357942271"
       rpy="0 1.3963 0" />
     <parent
@@ -68,4 +68,32 @@
         xyz="0 0 0" />
   </joint>
+  <link name="camera1_calib">
+    </link>
+  <joint name="camera1_calib_joint"
+      type="fixed">
+      <origin
+        xyz="0.768379569054 0.148829653859 0.454491734505"
+        rpy="0 0 0 " />
+      <parent
+        link="base_link" />
+      <child
+        link="camera1_calib" />
+      <axis
+        xyz="0 0 0" />
+  </joint>
+  <link name="camera_link">
+    </link>
+  <joint name="orbbec_joint"
+      type="fixed">
+      <origin
+        xyz="0.0 0.023878177 0.0"
+        rpy="0 1.3963 0" />
+      <parent
+        link="camera1_calib" />
+      <child
+        link="camera_link" />
+      <axis
+        xyz="0 0 0" />
+  </joint>
   <gazebo reference="camera1_link">
       <material>Gazebo/Black</material>
@@ -83,5 +111,5 @@
               </image>
               <clip>
-                  <near>0.3</near>
+                  <near>0.1</near>
                   <far>5.0</far>
               </clip>

File: ros2_ws/src/wetexplorer/wetexplorer_description/urdf/gazebo.xacro (robot description, xacro)
@@ -9,5 +9,5 @@
             <joint_name>sprocket_right_joint</joint_name>
             <joint_name>sprocket_left_joint</joint_name>
-            <!-- <joint_name>lift_joint</joint_name>               -->
+            <joint_name>lift_joint</joint_name>
         </plugin>
     </gazebo>

Commit message: update: change gps URDF to match new robot design

File: ros2_ws/src/wetexplorer/wetexplorer_description/urdf/accesories/gps.xacro (robot description, xacro)
@@ -104,4 +104,19 @@
       xyz="0 0 0" />
   </joint>
+  <link
+    name="gps">
+  </link>
+  <joint name="gps_joint2"
+    type="fixed">
+    <origin
+      xyz="00.10541 0.3 0.53942"
+      rpy="0 0 0" />
+    <parent
+      link="base_link" />
+    <child
+      link="gps" />
+    <axis
+      xyz="0 0 0" />
+  </joint>
   <gazebo reference="gps_frame_link">
       <material>Gazebo/LightGrey</material>
